File: coughgui/circuit/lcdmicrpi/lcdmicrpi.kicad_pcb (KiCad board)
At the start: 2 copper layers, 32.4 x 76.4 mm, 7 parts

Commit message: pcb shield
Routing:
- added copper zone on B.Cu, net (none)
- added copper zone on F.Cu, net (none)

Commit message: Project Stetoskop
Other:
- net class Default removed
